Commit message: dialing in

File: dingo_ws/src/jax_description/urdf/jax.urdf (robot description, URDF)
Before this commit: robot dingo, 17 links, 16 joints
Links:
- link FL_link1: geometry collision mesh filename=package://jax_description/meshes/L_link1_collision.STL; visual mesh filename=package://jax_description/meshes/FL_link1.dae
- link FL_link2: geometry collision mesh filename=package://jax_description/meshes/L_link2_collision.STL; visual mesh filename=package://jax_description/meshes/L_link2.dae
- link FL_link3: geometry collision mesh filename=package://jax_description/meshes/L_link3_collision.STL; visual mesh filename=package://jax_description/meshes/L_link3.dae
- link FL_link4: geometry collision mesh filename=package://jax_description/meshes/link4_collision.STL; visual mesh filename=package://jax_description/meshes/link4.dae
- link FR_link1: geometry collision mesh filename=package://jax_description/meshes/R_link1_collision.STL; visual mesh filename=package://jax_description/meshes/FR_link1.dae
- link FR_link2: geometry collision mesh filename=package://jax_description/meshes/R_link2_collision.STL; visual mesh filename=package://jax_description/meshes/R_link2.dae
- link FR_link3: geometry collision mesh filename=package://jax_description/meshes/R_link3_collision.STL; visual mesh filename=package://jax_description/meshes/R_link3.dae
- link FR_link4: geometry collision mesh filename=package://jax_description/meshes/link4_collision.STL; visual mesh filename=package://jax_description/meshes/link4.dae
- link RL_link1: geometry collision mesh filename=package://jax_description/meshes/L_link1_collision.STL; visual mesh filename=package://jax_description/meshes/RL_link1.dae
- link RL_link2: geometry collision mesh filename=package://jax_description/meshes/L_link2_collision.STL; visual mesh filename=package://jax_description/meshes/L_link2.dae
- link RL_link3: geometry collision mesh filename=package://jax_description/meshes/L_link3_collision.STL; visual mesh filename=package://jax_description/meshes/L_link3.dae
- link RL_link4: geometry collision mesh filename=package://jax_description/meshes/link4_collision.STL; visual mesh filename=package://jax_description/meshes/link4.dae
- link RR_link1: geometry collision mesh filename=package://jax_description/meshes/R_link1_collision.STL; visual mesh filename=package://jax_description/meshes/RR_link1.dae
- link RR_link2: geometry collision mesh filename=package://jax_description/meshes/R_link2_collision.STL; visual mesh filename=package://jax_description/meshes/R_link2.dae
- link RR_link3: geometry collision mesh filename=package://jax_description/meshes/R_link3_collision.STL; visual mesh filename=package://jax_description/meshes/R_link3.dae
- link RR_link4: geometry collision mesh filename=package://jax_description/meshes/link4_collision.STL; visual mesh filename=package://jax_description/meshes/link4.dae
- link base_link: geometry collision mesh filename=package://jax_description/meshes/base_collision.STL; visual mesh filename=package://jax_description/meshes/base_link.dae
